File: eagle/MainPCB/avocado-rev01/avocado-rev01_3.sch (KiCad schematic (older format))
At the start: 29 parts, among them J1 10118194-0001LF, J3 0475710001, P2 camconn, U1 V3S, X1 XTAL3.2X2, X2 XTAL5X1.9

Commit message: better routing v2
Connections:
- net USB-: now reaches J1.2 (DM), U1.110 (USB-DM)
- net USB+: now reaches J1.3 (DP), U1.111 (USB-DP)
Changed lines of the file:
@@
 EESchema Schematic File Version 4
+LIBS:avocado-rev01-cache
 EELAYER 29 0
 EELAYER END
@@
 Text Label 3100 6100 0    50   ~ 0
 CK_P
+Text Label 2800 4000 0    50   ~ 0
+USB+
+Text Label 2850 3900 0    50   ~ 0
+USB-
 $EndSCHEMATC
