File: eagle/MainPCB/avocado-rev01.ODL.sch (EAGLE design)
At the start: 141 parts, among them IC1 1V8, IC2 3V#, IC3 1V2, J1 10118194-0001LF, J3 0475710001, P2 CONNECTOR-15686115148922, U1 V3S, U2 AP65111A, U3 AP65111A, U4 AP65111A, U5 PMIC-LDO-XC6206P302MR(SOT23)

Commit message: updated
Parts:
- removed C69, C73: 4u7, marius:C0603
- removed C70, C74: 47p, marius:C0603
- removed C71, C72, C75, C76: 10u, marius:C0603
- removed D3: LL-R3528RGBC-008-B, LL-R3528RGBC-008-B:LL-R3528RGBC-008-B
- removed IC1: 1V8, AP3410:MCP73811/2
- removed IC2: 3V#, AP3410:MCP73811/2
- removed IC3: 1V2, AP3410:MCP73811/2
- removed L7, L8: 2.2uH-DCR<0.1R-1.5A, marius:L4X4
- removed R40: 470K-1%, resistor:R-EU_R0402
- removed R41, R43: 100K-1%, resistor:R-EU_R0402
- removed R42: 200K-1%, resistor:R-EU_R0402
- removed R44, R45, R46: (no value), resistor:R-EU_R0402
- removed SJ1, SJ2, SJ3: (no value), jumper:SJ
- added C50, C56, C57, C59, C64: 4u7, marius:C0603
- added C51, C52, C53, C60, C61, C62, C63: 10u, marius:C0603
- added C54, C55: 1n, marius:C0603
- added C58, C65, C66, C67, C68: 1u, marius:C0603
- added CN1: (no value), adafruit:JST_2PIN-SMT-RA
- added L5, L6: 2.2uH-DCR<0.1R-1.5A, marius:L6X6
- added R33: 0R03, resistor:R-EU_R1206
- added R34: 47k, resistor:R-EU_R0402
- added R35: 1K, resistor:R-EU_R0402
- added R36: 1k, resistor:R-EU_R0402
- added R37, R38: 0R, resistor:R-EU_R0402
- added R39: 0R NC, resistor:R-EU_R0402
- added SW1: SPST_TACT-KMR2, adafruit:SPST_TACT-KMR2
- added U6: AXP209, AXP209:AXP209
- C1, C2, C3, C4: device marius:C0402 -> marius:C0603
- C46: value 4u7 -> 1u
- C47: value 47p -> 4u7
- C48, C49: value 10u -> 4u7
- L4: device marius:L4X4 -> marius:L6X6
- R1, R17, R18, R19, R2, R20, R21, R22, R23, R24, R25, R26, R27, R28, R29, R3, R30: device resistor:R-EU_R0402 -> resistor:R-EU_R0603
- R31: value 100K-1% -> 200K-1%
- R32: value 100K-1% -> 100R-1%
Connections:
- removed net LEDD: J3.DET, R44.1
- removed net N$33: IC1.LX, L8.1
- removed net N$35: IC2.LX, L7.1
- removed net N$36: C70.1, IC2.FB, R40.1, R41.1
- removed net N$37: C74.1, IC1.FB, R42.1, R43.1
- removed net N$38: D3.CATHODE_RED, R46.2
- removed net N$39: D3.CATHODE_GREEN, R45.2
- removed net N$41: D3.CATHODE_BLUE, R44.2
- new net ACIN-5V: C52.2, R39.2, U6.ACIN
- new net CHGLED: U6.CHGLED
- new net DC21V2: C55.2, C61.2, L4.2, U6.DCDC2
- new net DC31V2: C54.2, C62.2, L5.2, U6.DCDC3
- new net IPSOUT: C49.1, C53.2, C59.1, C60.1, C63.2, C64.2, U6.APS, U6.IPSOUT, U6.LDO24IN, U6.LDO3IN, U6.VIN1, U6.VIN2, U6.VIN3
- new net LDO13V3: C46.1, U6.LDO1
- new net LDO1V8: C48.1, U6.LDO3
- new net LDO3V: C47.1, U6.LDO2
- new net LDO42V8: C50.1, U6.LDO4
- new net N$26: L5.1, U6.LX3
- new net N$32: R34.1
- new net N$40: U6.LDO1SET
- new net N$51: C67.2, R34.2, U6.PWROK
- new net N$52: R37.1, U6.SDA
- new net N$62: C56.1, C58.1, L6.2, R33.1, U6.CHSENSE
- new net N$64: R38.1, U6.SCK
- new net N$67: R32.2, U6.TS
- new net N$73: R31.2, U6.BIAS
- new net N$75: C68.1, R36.1, U6.PWRON
- new net N$76: R35.1, U6.N_OE
- new net N$78: C66.2, U6.VREF
- new net N$79: C65.2, U6.VINT
- new net N$81: R36.2, SW1.S1
- new net NMI_N: U6.IRQ/WAKEUP
- new net USB0_DRV: U6.N_VBUSEN
- new net USBVBUS: C51.2, R39.1, U6.VBUS
- new net VBAT: C57.1, C58.2, CN1.2, R33.2, U6.BAT, U6.BATSENSE
- net 1V2: no longer C46.2, C47.2, C48.2, L4.2, R31.2
- net 1V8: no longer C73.2, C74.2, C75.2, L8.2, R42.2
- net 3V3: now also J3.VSS; no longer C69.2, C70.2, C71.2, D3.COMM_ANODE, L7.2, R40.2
- net GND: now also C46.2, C47.2, C48.2, C50.2, C51.1, C52.1, C53.1, C54.1, C55.1, C56.2, C57.2, C59.2, C60.2, C61.1, C62.1, C63.1, C64.1, C65.1, C66.1, C67.1, C68.2, CN1.1, R31.1, R32.1, R35.2, SW1.P1, U6.AGND, U6.EP, U6.PGND1, U6.PGND2, U6.PGND3; no longer C46.1, C48.1, C69.1, C71.1, C72.2, C73.1, C75.1, C76.2, IC1.GND, IC2.GND, IC3.GND, J3.VSS, R32.2, R41.2, R43.2
- net LED0: no longer R45.1
- net LED1: no longer R46.1
- net N$7: now also U6.LX2; no longer IC3.LX
- net N$8: now also L6.1, U6.LX1; no longer C47.1, IC3.FB, R31.1, R32.1
- net SCL: now also R38.2
- net SDA: now also R37.2
- net VCC: no longer C49.1, C72.1, C76.1, IC1.VIN, IC2.VIN, IC3.VIN
