File: eagle/MainPCB/avocado-rev01.OLD.brd (EAGLE design)
At the start: 60 x 60 mm, 141 parts, among them IC1 1V8, IC2 3V#, IC3 1V2, J1 10118194-0001LF, J3 0475710001, P2 CONNECTOR-15686115148922, U1 V3S, U2 AP65111A, U3 AP65111A, U4 AP65111A, U5 PMIC-LDO-XC6206P302MR(SOT23)

Commit message: updated
Parts:
- removed C69, C73: 4u7, marius:C0603
- removed C70, C74: 47p, marius:C0603
- removed C71, C72, C75, C76: 10u, marius:C0603
- removed D3: LL-R3528RGBC-008-B, LL-R3528RGBC-008-B:LED_LL-R3528RGBC-008-B
- removed IC1: 1V8, AP3410:SOT23-5L
- removed IC2: 3V#, AP3410:SOT23-5L
- removed IC3: 1V2, AP3410:SOT23-5L
- removed L7, L8: 2.2uH-DCR<0.1R-1.5A, marius:ASPI-4030S-253675
- removed R40: 470K-1%, resistor:R0402
- removed R41, R43: 100K-1%, resistor:R0402
- removed R42: 200K-1%, resistor:R0402
- removed R44, R45, R46: (no value), resistor:R0402
- removed SJ1, SJ2, SJ3: (no value), jumper:SJ
- added C50, C56, C57, C59, C64: 4u7, marius:C0603
- added C51, C52, C53, C60, C61, C62, C63: 10u, marius:C0603
- added C54, C55: 1n, marius:C0603
- added C58, C65, C66, C67, C68: 1u, marius:C0603
- added CN1: (no value), adafruit:JST-PH-2-SMT-RA
- added L5, L6: 2.2uH-DCR<0.1R-1.5A, marius:B82462A4153K
- added R33: 0R03, resistor:R1206
- added R34: 47k, resistor:R0402
- added R35: 1K, resistor:R0402
- added R36: 1k, resistor:R0402
- added R37, R38: 0R, resistor:R0402
- added R39: 0R NC, resistor:R0402
- added SW1: SPST_TACT-KMR2, adafruit:KMR2
- added U6: AXP209, AXP209:QFN40P600X600X80-49N
- C1, C2, C3, C4: device marius:C0402 -> marius:C0603
- C46: value 4u7 -> 1u
- C47: value 47p -> 4u7
- C48, C49: value 10u -> 4u7
- L4: device marius:ASPI-4030S-253675 -> marius:B82462A4153K
- R1, R17, R18, R19, R2, R20, R21, R22, R23, R24, R25, R26, R27, R28, R29, R3, R30: device resistor:R0402 -> resistor:R0603
- R31: value 100K-1% -> 200K-1%
- R32: value 100K-1% -> 100R-1%
- moved R32 62.2 mm to (-35.8, 35.2)
- moved R31 55.4 mm to (-35.8, 32.8)
- moved L4 45.1 mm to (-11.0, 6.84), turned to 90 degrees
- moved C23 44.2 mm to (-25.8, 17.2)
- moved C27 44.2 mm to (-25.8, 11.2)
- moved C32 44.2 mm to (-18.4, 11.2)
- moved C36 44.2 mm to (-18.2, 16.2)
- moved C37 44.2 mm to (-18.2, 18.2)
- moved C45 44.2 mm to (-36.4, 11.6)
- moved U5 44.2 mm to (-37.4, 25.4)
- moved C22 44.2 mm to (-25.6, 18.8)
- moved C24 44.2 mm to (-25.6, 15.8)
- moved C25 44.2 mm to (-25.8, 14.4)
- moved C26 44.2 mm to (-26.0, 12.6)
- moved C28 44.2 mm to (-25.6, 9.40)
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Connections:
- removed net LEDD: J3.11, R44.1
- removed net N$33: IC1.3, L8.P$1
- removed net N$35: IC2.3, L7.P$1
- removed net N$36: C70.1, IC2.5, R40.1, R41.1
- removed net N$37: C74.1, IC1.5, R42.1, R43.1
- removed net N$38: D3.2, R46.2
- removed net N$39: D3.3, R45.2
- removed net N$41: D3.4, R44.2
- new net ACIN-5V: C52.2, R39.2, U6.32, U6.33
- new net CHGLED: U6.36
- new net DC21V2: C55.2, C61.2, L4.P$2, U6.10
- new net DC31V2: C54.2, C62.2, L5.P$2, U6.17
- new net IPSOUT: C49.1, C53.2, C59.1, C60.1, C63.2, C64.2, U6.13, U6.14, U6.21, U6.34, U6.35, U6.40, U6.44, U6.7
- new net LDO13V3: C46.1, U6.28
- new net LDO1V8: C48.1, U6.41
- new net LDO3V: C47.1, U6.12
- new net LDO42V8: C50.1, U6.11
- new net N$26: L5.P$1, U6.15
- new net N$32: R34.1
- new net N$40: U6.27
- new net N$51: C67.2, R34.2, U6.25
- new net N$52: R37.1, U6.1
- new net N$62: C56.1, C58.1, L6.P$2, R33.1, U6.43
- new net N$64: R38.1, U6.2
- new net N$67: R32.2, U6.37
- new net N$73: R31.2, U6.23
- new net N$75: C68.1, R36.1, U6.47
- new net N$76: R35.1, U6.4
- new net N$78: C66.2, U6.24
- new net N$79: C65.2, U6.26
- new net N$81: R36.2, SW1.4
- new net NMI_N: U6.48
- new net USB0_DRV: U6.6
- new net USBVBUS: C51.2, R39.1, U6.31
- new net VBAT: C57.1, C58.2, CN1.1, R33.2, U6.38, U6.39, U6.42
- net 1V2: no longer C46.2, C47.2, C48.2, L4.P$2, R31.2
- net 1V8: no longer C73.2, C74.2, C75.2, L8.P$2, R42.2
- net 3V3: now also J3.6; no longer C69.2, C70.2, C71.2, D3.1, L7.P$2, R40.2
- net GND: now also C46.2, C47.2, C48.2, C50.2, C51.1, C52.1, C53.1, C54.1, C55.1, C56.2, C57.2, C59.2, C60.2, C61.1, C62.1, C63.1, C64.1, C65.1, C66.1, C67.1, C68.2, CN1.2, R31.1, R32.1, R35.2, SW1.3, U6.16, U6.22, U6.46, U6.49, U6.9; no longer C46.1, C48.1, C69.1, C71.1, C72.2, C73.1, C75.1, C76.2, IC1.2, IC2.2, IC3.2, J3.6, R32.2, R41.2, R43.2
- net LED0: no longer R45.1
- net LED1: no longer R46.1
- net N$7: now also U6.8; no longer IC3.3
- net N$8: now also L6.P$1, U6.45; no longer C47.1, IC3.5, R31.1, R32.1
- net SCL: now also R38.2
- net SDA: now also R37.2
- net VCC: no longer C49.1, C72.1, C76.1, IC1.4, IC2.4, IC3.4
Routing:
- net N$24: track 0.21 -> 12.8 mm
- net GND: track 23.9 -> 13.9 mm
- net N$10: track 0.00 -> 9.29 mm
- net N$11: track 0.00 -> 8.04 mm
- net N$9: track 0.00 -> 7.30 mm
- net N$14: track 0.53 -> 7.29 mm
- net 3V3: track 30.9 -> 36.9 mm
- net N$12: track 0.00 -> 5.30 mm
- net VCC: track 55.9 -> 51.2 mm
- net N$36: track 2.52 -> 0.00 mm
- net N$35: track 2.03 -> 0.00 mm
- removed copper zone on layer 1, net VCC
Other:
- board text removed: "OBS! 0402 capacitors"
