File: eagle/MainPCB/avocado-rev01.brd (EAGLE design)
At the start: 60 x 60 mm, 141 parts, among them IC1 1V8, IC2 3V#, IC3 1V2, J1 10118194-0001LF, J3 0475710001, P2 CONNECTOR-15686115148922, U1 V3S, U2 AP65111A, U3 AP65111A, U4 AP65111A, U5 PMIC-LDO-XC6206P302MR(SOT23)

Commit message: added jumpers
Parts:
- removed C46, C73: 4u7, marius:C0603
- removed C47, C74: 47p, marius:C0603
- removed C48, C49, C75, C76: 10u, marius:C0603
- removed IC1: 1V8, AP3410:SOT23-5L
- removed IC3: 1V2, AP3410:SOT23-5L
- removed L4, L8: 2.2uH-DCR<0.1R-1.5A, marius:ASPI-4030S-253675
- removed R31, R32, R43: 100K-1%, resistor:R0402
- removed R42: 200K-1%, resistor:R0402
- removed SJ2, SJ3: (no value), jumper:SJ
- added C54, C58: 4u7, marius:C0603
- added C55, C59: 47p, marius:C0603
- added C56, C57, C60, C61: 10u, marius:C0603
- added IC5, IC6: 3V#, AP3410:SOT23-5L
- added L6, L9: 2.2uH-DCR<0.1R-1.5A, marius:ASPI-4030S-253675
- added R35, R36, R38: 100K-1%, resistor:R0402
- added R37: 200K-1%, resistor:R0402
- added SJ4, SJ5, SJ6, SJ8, SJ9: (no value), jumper:SJ
- moved SJ1 150.6 mm to (63.4, 17.8), turned to 90 degrees
- moved U5 126.7 mm to (47.0, 23.8), turned to 270 degrees
- moved C22 111.4 mm to (44.2, 23.8), turned to 90 degrees
- moved C23 109.8 mm to (42.6, 23.8), turned to 90 degrees
- moved L7 81.6 mm to (68.0, 13.2), turned to 90 degrees
- moved C69 79.6 mm to (65.2, 13.8), turned to 90 degrees
- moved R41 79.2 mm to (70.0, 9.00), turned to 90 degrees
- moved C70 78.4 mm to (68.8, 5.40), turned to 270 degrees
- moved C71 77.7 mm to (63.6, 13.8), turned to 90 degrees
- moved R40 77.6 mm to (70.0, 5.60), turned to 270 degrees
- moved IC2 77.2 mm to (68.0, 9.00), turned to 180 degrees
- moved C72 74.6 mm to (65.8, 8.60), turned to 90 degrees
- moved R3 50.0 mm to (112.8, 40.8)
- moved R18 49.0 mm to (111.6, 45.0)
- moved R17 47.9 mm to (112.8, 45.0)
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Connections:
- removed net N$33: IC1.3, L8.P$1
- removed net N$37: C74.1, IC1.5, R42.1, R43.1
- removed net N$7: IC3.3, L4.P$1
- removed net N$8: C47.1, IC3.5, R31.1, R32.1
- new net N$45: IC5.3, L6.P$1
- new net N$46: C55.1, IC5.5, R35.1, R36.1
- new net N$51: IC6.3, L9.P$1
- new net N$52: C59.1, IC6.5, R37.1, R38.1
- new net P1V2: C18.1, C19.1, L3.P$2, R14.1, SJ6.1
- new net P1V8: C13.1, C14.1, L2.P$2, R10.1, SJ5.1
- new net P3V3: C8.1, C9.1, L1.P$2, R6.1, SJ4.1
- new net PRE1V2: C54.2, C55.2, C56.2, L6.P$2, R35.2, SJ8.1
- new net PRE1V8: C58.2, C59.2, C60.2, L9.P$2, R37.2, SJ9.1
- new net PRE3V3: C69.2, C70.2, C71.2, L7.P$2, R40.2, SJ1.1
- net 1V2: now also SJ6.2, SJ8.2; no longer C18.1, C19.1, C46.2, C47.2, C48.2, L3.P$2, L4.P$2, R14.1, R31.2
- net 1V8: now also SJ5.2, SJ9.2; no longer C13.1, C14.1, C73.2, C74.2, C75.2, L2.P$2, L8.P$2, R10.1, R42.2
- net 3V3: now also SJ1.2, SJ4.2; no longer C69.2, C70.2, C71.2, C8.1, C9.1, L1.P$2, L7.P$2, R40.2, R6.1
- net GND: now also C54.1, C56.1, C57.2, C58.1, C60.1, C61.2, IC5.2, IC6.2, R36.2, R38.2; no longer C46.1, C48.1, C49.2, C73.1, C75.1, C76.2, IC1.2, IC3.2, R32.2, R43.2
- net VCC: now also C57.1, C61.1, IC2.1, IC5.1, IC5.4, IC6.1, IC6.4; no longer C49.1, C76.1, IC1.4, IC3.4
Routing:
- net 3V3: track 30.9 -> 6.40 mm, vias 2 -> 0
- net P1V8: track 0.00 -> 16.1 mm, vias 0 -> 2
- net P1V2: track 0.00 -> 16.1 mm, vias 0 -> 2
- net 1V8: track 16.1 -> 0.00 mm, vias 2 -> 0
- net 1V2: track 16.1 -> 0.00 mm, vias 2 -> 0
- net P3V3: track 0.00 -> 15.2 mm, vias 0 -> 2
- net PRE3V3: track 0.00 -> 13.8 mm
- net PRE1V8: track 0.00 -> 13.8 mm
- net PRE1V2: track 0.00 -> 13.8 mm
- net VCC: track 55.9 -> 68.1 mm, vias 6 -> 12
- net GND: track 23.9 -> 34.0 mm
- net N$52: track 0.00 -> 4.03 mm
- net N$46: track 0.00 -> 4.03 mm
- net N$51: track 0.00 -> 2.03 mm
- net N$45: track 0.00 -> 2.03 mm
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Other:
- board size 60 x 60 mm -> 100 x 60 mm

Commit message: high
Parts:
- moved RX1 36.9 mm to (72.6, 65.4), turned to 270 degrees
- moved TX1 34.2 mm to (70.6, 65.4), turned to 270 degrees
- moved TX2 31.6 mm to (68.6, 65.4), turned to 0 degrees
- moved RX2 29.0 mm to (66.6, 65.4), turned to 270 degrees
- moved R27 28.5 mm to (97.2, 63.2)
- moved R28 28.5 mm to (95.2, 63.2)
- moved R29 28.5 mm to (93.2, 63.2)
- moved R30 28.5 mm to (91.2, 63.2)
- moved PWM0 26.5 mm to (64.6, 65.4), turned to 270 degrees
- moved C20 25.0 mm to (-20.2, 56.4)
- moved PWM1 24.1 mm to (62.6, 65.4), turned to 270 degrees
- moved SCL0 21.7 mm to (60.6, 65.4), turned to 270 degrees
- moved SDA0 19.5 mm to (58.6, 65.4), turned to 270 degrees
- moved C1 19.1 mm to (-8.80, 52.8)
- moved C2 19.1 mm to (-4.80, 52.8)
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Connections:
- net N$5 renamed USBDIFF_N
- net N$6 renamed USBDIFF_P
- net N$65 renamed D0_N
- net N$66 renamed D0_P
- net N$68 renamed D1_N
- net N$69 renamed D1_P
- net N$70 renamed CK_P
- net N$72 renamed CK_N
Routing:
- net CK_P: track 0.00 -> 2.21 mm, vias 0 -> 1
- net CK_N: track 0.00 -> 2.21 mm, vias 0 -> 1
- net USBDIFF_N: track 0.86 -> 0.00 mm
- net USBDIFF_P: track 0.86 -> 0.00 mm

Commit message: working
Parts:
- moved C3 12.3 mm to (36.9, 56.2)
- moved C4 12.3 mm to (36.9, 50.2)
- moved X1 12.3 mm to (36.9, 53.2)
Routing:
- net D0_P: track 0.00 -> 32.6 mm, vias 0 -> 1
- net D0_N: track 0.00 -> 32.1 mm, vias 0 -> 1
- net D1_P: track 0.00 -> 28.5 mm, vias 0 -> 1
- net D1_N: track 0.00 -> 28.0 mm, vias 0 -> 1
- net CK_N: track 2.21 -> 25.1 mm
- net CK_P: track 2.21 -> 24.6 mm
- net SDC0_D2: track 0.00 -> 20.9 mm
- net SDC0_D3: track 0.00 -> 20.6 mm
- net SDC0_D1: track 0.00 -> 20.4 mm
- net SDC0_CMD: track 0.00 -> 19.8 mm
- net SDC0_CLK: track 0.00 -> 19.8 mm
- net SDC0_D0: track 0.00 -> 19.7 mm
- added copper zone on layer 1, net N$26
- added copper zone on layer 16, net N$32
- added copper zone on layer 3, net N$5
- added copper zone on layer 2, net N$6
- added copper zone on layer 2, net N$7
- added copper zone on layer 3, net N$8

Commit message: In progress
Parts:
- R16: device marius:R0603 -> marius:R0402
- moved C25 45.5 mm to (-19.1, 28.1)
- moved C27 45.5 mm to (-19.1, 24.9)
- moved C39 45.5 mm to (-27.1, 42.9)
- moved C40 45.5 mm to (-27.1, 41.3)
- moved C41 45.5 mm to (-27.1, 40.1)
- moved C42 45.5 mm to (-27.1, 39.1)
- moved C24 45.5 mm to (-18.9, 29.5)
- moved C28 45.5 mm to (-18.9, 23.1)
- moved C30 45.5 mm to (-11.2, 22.3)
- moved C32 45.5 mm to (-11.7, 24.9)
- moved C33 45.5 mm to (-13.2, 37.7)
- moved C43 45.5 mm to (-24.6, 37.5)
- moved C44 45.5 mm to (-25.6, 33.7)
- moved C45 45.5 mm to (-29.9, 35.5)
- moved C26 45.5 mm to (-19.2, 26.3)
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Connections:
- new net LEDD0: R45.1
- new net LEDD1: R46.1
- net LED0: no longer R45.1
- net LED1: no longer R46.1
Routing:
- net 3V3: track 6.40 -> 38.6 mm, vias 0 -> 9
- net USBDIFF_P: track 0.00 -> 26.0 mm
- net USBDIFF_N: track 0.00 -> 26.0 mm
- net N$4: track 0.00 -> 21.2 mm
- net N$3: track 0.00 -> 20.8 mm
- net CK_P: track 24.6 -> 34.5 mm
- net N$24: track 0.21 -> 9.78 mm
- net N$41: track 0.00 -> 9.48 mm
- net N$11: track 0.00 -> 9.46 mm
- net N$2: track 0.00 -> 9.44 mm
- net CK_N: track 25.1 -> 34.5 mm
- net N$1: track 0.00 -> 9.00 mm
- net D1_N: track 28.0 -> 33.9 mm
- net D1_P: track 28.5 -> 33.9 mm
- net N$14: track 0.00 -> 5.25 mm
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- added copper zone on layer 16, net 1V2
- added copper zone on layer 16, net 1V8
- added copper zone on layer 16, net 3V3
- added copper zone on layer 3, net 3V3
- added copper zone on layer 2, net GND
- added copper zone on layer 1, net N$64
- added copper zone on layer 1, net N$65
- added copper zone on layer 16, net VCC

Commit message: In progress
Parts:
- removed C40, C43: 10u, marius:C0603
- added 3V3: 10u, marius:C0603
- moved C45 63.4 mm to (33.5, 36.7), turned to 0 degrees
- moved C44 59.2 mm to (33.5, 34.6), turned to 0 degrees
- moved C39 52.5 mm to (22.1, 24.2), turned to 0 degrees
- moved C55 50.6 mm to (30.8, 5.00)
- moved C57 50.6 mm to (27.8, 8.20)
- moved C56 50.6 mm to (25.6, 13.4)
- moved SJ8 50.6 mm to (25.4, 17.4)
- moved C54 50.6 mm to (27.2, 13.4)
- moved IC5 50.6 mm to (30.0, 8.60)
- moved L6 50.6 mm to (30.0, 12.8)
- moved R35 50.6 mm to (32.0, 5.20)
- moved R36 50.6 mm to (32.0, 8.60)
- moved C42 48.7 mm to (21.6, 38.1), flipped to the bottom, turned to 270 degrees
- moved C41 47.6 mm to (19.0, 28.0), flipped to the bottom
- moved C25 46.3 mm to (26.9, 33.4), flipped to the bottom, turned to 0 degrees
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Connections:
- net 3V3: now also 3V3.1; no longer C40.1, C43.1
- net GND: now also 3V3.2; no longer C40.2, C43.2
Routing:
- net 1V2: track 0.00 -> 94.0 mm, vias 0 -> 26
- net 1V8: track 0.00 -> 61.0 mm, vias 0 -> 17
- net 3V: track 3.38 -> 27.8 mm, vias 0 -> 3
- net 3V3: track 38.6 -> 58.3 mm, vias 9 -> 28
- net GND: track 38.5 -> 50.7 mm, vias 11 -> 42
- net VCC: track 67.9 -> 75.4 mm
- net 3V1: track 4.51 -> 0.00 mm, vias 6 -> 0
- net N$1: track 9.00 -> 13.4 mm
- net N$2: track 9.44 -> 13.7 mm
- net USB-ID: track 0.00 -> 2.75 mm
- added copper zone on layer 1, net GND1
- added copper zone on layer 1, net GND2

Commit message: in progress
Parts:
- moved RX1 30.0 mm to (52.2, 24.3), turned to 180 degrees
- moved TX1 27.1 mm to (52.2, 26.3), turned to 180 degrees
- moved D2 27.0 mm to (73.3, 24.9)
- moved R17 27.0 mm to (66.2, 24.9)
- moved R18 27.0 mm to (67.3, 24.9)
- moved R19 27.0 mm to (68.4, 24.9)
- moved TX2 24.3 mm to (52.2, 28.3), turned to 270 degrees
- moved D1 22.7 mm to (73.3, 30.4)
- moved R1 22.7 mm to (68.5, 30.2)
- moved R2 22.7 mm to (67.3, 30.2)
- moved R3 22.7 mm to (66.2, 30.2)
- moved D3 22.3 mm to (73.3, 35.8)
- moved R44 22.3 mm to (66.2, 35.8)
- moved R45 22.3 mm to (67.3, 35.8)
- moved R46 22.3 mm to (68.4, 35.8)
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Connections:
- removed net N$57: PWM0.1, U1.43
- removed net N$58: PWM1.1, U1.44
- net LEDD0: now also PWM0.1, U1.43
- net LEDD1: now also PWM1.1, U1.44
Routing:
- net SDA: track 0.00 -> 111.0 mm, vias 0 -> 1
- net SCL: track 0.00 -> 108.4 mm, vias 0 -> 1
- net LEDD: track 0.00 -> 95.6 mm, vias 0 -> 2
- net LED1: track 0.00 -> 56.1 mm
- net LED0: track 0.00 -> 55.5 mm
- net LED2: track 0.00 -> 54.3 mm
- net LED3: track 5.03 -> 57.8 mm, vias 0 -> 2
- net LED4: track 3.28 -> 55.9 mm, vias 0 -> 2
- net CAM_IO1: track 0.00 -> 44.0 mm
- net CAM_IO0: track 0.00 -> 42.1 mm
- net LEDD1: track 0.00 -> 41.7 mm
- net LEDD0: track 0.00 -> 40.1 mm
- net N$60: track 0.00 -> 37.5 mm
- net N$59: track 0.00 -> 37.5 mm
- net N$56: track 0.00 -> 27.3 mm
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- added copper zone on layer 3, net GND
- added copper zone on layer 2, net N$5
- removed copper zone on layer 3, net N$5

Commit message: in progress
Parts:
- moved R40 0.15 mm to (96.6, 4.50)
- moved R37 0.14 mm to (62.6, 5.05)
- moved R35 0.11 mm to (32.1, 5.15)
Routing:
- net GND: track 66.5 -> 68.8 mm, vias 58 -> 69
- added copper zone on layer 1, net P1V2
- added copper zone on layer 1, net P1V8
- added copper zone on layer 1, net P3V3
- added copper zone on layer 1, net PRE1V2
- added copper zone on layer 16, net PRE1V2
- added copper zone on layer 1, net PRE1V8
- added copper zone on layer 16, net PRE1V8
- added copper zone on layer 1, net PRE3V3
- added copper zone on layer 16, net PRE3V3

Commit message: In progress
Parts:
- moved R16 2.53 mm to (12.8, 40.8), turned to 180 degrees
Routing:
- net GND: track 68.8 -> 75.9 mm, vias 69 -> 71
- net N$13: track 2.48 -> 1.58 mm
- net 1V2: vias 26 -> 24
