File: eagle/MainPCB/avocado-rev01.brd (EAGLE design)
At the start: 100 x 60 mm, 143 parts, among them IC2 3V#, IC5 3V#, IC6 3V#, J1 10118194-0001LF, J3 0475710001, P2 CONNECTOR-15686115148922, U1 V3S, U2 AP65111A, U3 AP65111A, U4 AP65111A, U5 PMIC-LDO-XC6206P302MR(SOT23)

Commit message: drc
Parts:
- moved CAMIO0 3.76 mm to (43.0, 54.0)
- moved CAMIO1 3.76 mm to (41.0, 54.0)
Routing:
- net CAM_IO0: track 42.1 -> 57.6 mm, vias 0 -> 1
- net GND: track 75.9 -> 90.1 mm, vias 71 -> 83
- net CAM_IO1: track 44.0 -> 57.0 mm, vias 0 -> 1
- net 3V3: track 74.2 -> 81.4 mm, vias 29 -> 30
- net 1V2: track 98.2 -> 102.0 mm, vias 24 -> 26
- net 1V8: track 74.5 -> 76.1 mm
- net N$13: track 1.58 -> 2.41 mm
- net VCC: track 75.4 -> 75.9 mm
Other:
- board text removed: "OBS! 0402 capacitors"

Commit message: In Progress
Parts:
- added C40, C43, C46: 10u, marius:C0603
- added CLK, INT, RST, WOL: TEST_TESTPOINT, marius:TEST_TESTPOINT
- added J2: CONNECTOR-10HEADER-5X2, marius:HEADER-5X2
- added J4: CONNECTOR-4HEADER4, marius:HEADER-4
- added J5: CONNECTOR-3HEADER3, marius:HEADER-3
- added R31: 10k, resistor:R0402
- IC6: value 3V# -> (none)
Connections:
- removed net N$53: MISO.1, U1.52
- removed net N$54: SCK.1, U1.53
- removed net N$55: CS.1, U1.54
- removed net N$56: MOSI.1, U1.55
- new net CLK: CLK.1, J2.10
- new net CS: CS.1, J2.4, R31.2, U1.54
- new net INT: INT.1, J2.9
- new net MISO: J2.7, MISO.1, U1.52
- new net MOSI: J2.6, MOSI.1, U1.55
- new net RST: J2.3, RST.1
- new net SCK: J2.5, SCK.1, U1.53
- new net WOL: J2.8, WOL.1
- net 3V3: now also C43.1, J2.2, R31.1
- net GND: now also C40.1, C43.2, C46.1, J2.1, J4.1, J5.1
- net LEDD0: now also J5.2
- net SCL: now also J4.3
- net SDA: now also J4.4
- net VCC: now also C40.2, C46.2, J4.2, J5.3
Routing:
- net VCC: track 75.9 -> 136.4 mm
- net CS: track 0.00 -> 47.2 mm
- net SCK: track 0.00 -> 46.5 mm, vias 0 -> 1
- net MISO: track 0.00 -> 45.9 mm, vias 0 -> 1
- net LEDD0: track 40.1 -> 84.6 mm, vias 0 -> 1
- net MOSI: track 0.00 -> 41.5 mm
- net SDA: track 111.0 -> 151.3 mm, vias 1 -> 2
- net SCL: track 108.4 -> 148.6 mm, vias 1 -> 2
- net N$56: track 27.3 -> 0.00 mm
- net N$55: track 26.6 -> 0.00 mm
- net N$54: track 25.9 -> 0.00 mm
- net N$53: track 25.3 -> 0.00 mm
- net GND: track 90.1 -> 102.2 mm, vias 83 -> 86
- net RST: track 0.00 -> 11.6 mm
- net WOL: track 0.00 -> 11.0 mm
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- added copper zone on layer 1, net N$33
- added copper zone on layer 16, net N$33
- added copper zone on layer 2, net N$33

Commit message: In progress
Parts:
- added C47, C48: 10u, marius:C0603
- added J6: HR911105A, HR911105A:HANRUN_HR911105A
- added L4: 10uH(NC), marius:R0603
- added R32, R33, R34, R39: 51(NC), resistor:R0402
- added R42: 6K-1%, resistor:R0402
- moved R31 19.7 mm to (49.8, 47.8), turned to 45 degrees
Connections:
- new net ETH_RX_N: J6.6, R34.1, U1.89
- new net ETH_RX_P: J6.3, R33.1, U1.90
- new net ETH_TX_N: J6.2, R39.1, U1.91
- new net ETH_TX_P: J6.1, R32.1, U1.92
- new net N$37: R42.2, U1.94
- new net N$55: C47.1, J6.4, R32.2, R39.2
- new net N$56: C48.1, J6.5, L4.2, R33.2, R34.2
- net 3V3: now also C40.2, J4.2, L4.1
- net GND: now also C47.2, C48.2, J6.10, J6.11, J6.15, J6.16, J6.8, R42.1
- net LED3: now also J6.9
- net LED4: now also J6.12
- net VCC: no longer C40.2, J4.2
Routing:
- net VCC: track 136.4 -> 119.5 mm
- net 3V3: track 87.8 -> 89.9 mm, vias 31 -> 33
- net CS: track 47.2 -> 46.2 mm

Commit message: in progress
Parts:
- removed C43: 10u, marius:C0603
- removed CLK, INT, RST, WOL: TEST_TESTPOINT, marius:TEST_TESTPOINT
- removed J2: CONNECTOR-10HEADER-5X2, marius:HEADER-5X2
- added DIGITAL1, DIGITAL2, DIGITAL3, PB2, PB3: TEST_TESTPOINT, marius:TEST_TESTPOINT
- added SW1, SW2, SW3: SPST_TACT-KMR2, adafruit:KMR2
- moved L4 55.2 mm to (68.8, 46.5)
- moved C48 53.1 mm to (68.8, 48.2)
- moved R39 51.7 mm to (68.8, 43.2)
- moved R34 50.9 mm to (68.8, 49.8)
- moved C47 50.3 mm to (68.8, 44.8)
- moved R32 49.0 mm to (68.8, 52.2)
- moved R33 48.9 mm to (68.8, 51.0)
- moved R42 32.8 mm to (11.8, 44.2)
- moved CAMIO0 32.6 mm to (10.7, 58.7)
- moved CAMIO1 32.6 mm to (8.70, 58.7)
- moved C40 29.7 mm to (90.3, 54.1)
- moved J4 29.7 mm to (87.5, 57.1)
- moved J6 28.6 mm to (57.5, 53.5), flipped to the bottom, turned to 0 degrees
- moved SCK 21.8 mm to (38.3, 29.5), turned to 0 degrees
- moved CS 21.6 mm to (38.3, 31.8), turned to 0 degrees
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Connections:
- removed net CLK: CLK.1, J2.10
- removed net INT: INT.1, J2.9
- removed net RST: J2.3, RST.1
- removed net WOL: J2.8, WOL.1
- new net N$54: PB2.1, SW2.1, U1.41
- new net N$57: PB3.1, U1.42
- new net N$58: DIGITAL1.1, SW3.1, U1.2
- new net N$61: DIGITAL2.1, SW1.1, U1.1
- new net N$62: DIGITAL3.1, U1.128
- net 3V3: no longer C43.1, J2.2
- net CS: no longer J2.4
- net GND: now also SW1.2, SW2.2, SW3.2; no longer C43.2, J2.1
- net MISO: no longer J2.7
- net MOSI: no longer J2.6
- net SCK: no longer J2.5
Routing:
- net N$61: track 0.00 -> 106.0 mm
- net N$58: track 0.00 -> 104.6 mm
- net N$62: track 0.00 -> 98.1 mm
- net ETH_RX_P: track 0.00 -> 78.7 mm, vias 0 -> 1
- net ETH_TX_P: track 0.00 -> 77.3 mm
- net ETH_TX_N: track 0.00 -> 76.3 mm, vias 0 -> 1
- net N$54: track 0.00 -> 75.8 mm, vias 0 -> 4
- net ETH_RX_N: track 0.00 -> 74.6 mm, vias 0 -> 1
- net N$57: track 0.00 -> 67.5 mm, vias 0 -> 4
- net LED3: track 57.8 -> 116.3 mm
- net LED4: track 55.9 -> 103.1 mm, vias 2 -> 3
- net SCK: track 46.5 -> 12.7 mm, vias 1 -> 0
- net MOSI: track 41.5 -> 9.21 mm
- net MISO: track 45.9 -> 13.9 mm, vias 1 -> 0
- net CS: track 46.2 -> 14.3 mm
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- added copper zone on layer 1, net N$40

Commit message: in progress
Parts:
- moved SW2 4.01 mm to (94.8, 36.0)
- moved SW1 1.77 mm to (94.8, 41.2)
- moved SW3 0.79 mm to (94.8, 46.8)
Routing:
- net CK_N: track 41.1 -> 43.2 mm
- net CK_P: track 41.1 -> 43.2 mm
- net D0_N: track 41.3 -> 43.5 mm
- net D1_P: track 41.1 -> 43.0 mm
- net D1_N: track 41.1 -> 43.0 mm
- net D0_P: track 41.8 -> 43.5 mm
- net N$54: track 75.8 -> 74.7 mm
- net 3V: track 47.0 -> 46.0 mm
- net 1V2: track 102.0 -> 101.0 mm
- net P1V8: track 16.1 -> 15.2 mm
- net GND: track 112.9 -> 113.7 mm
- net N$61: track 106.0 -> 106.7 mm
- net N$58: track 104.6 -> 104.1 mm
