File: eagle/MainPCB/avocado-rev01.sch (EAGLE design)
At the start: 141 parts, among them IC1 1V8, IC2 3V#, IC3 1V2, J1 10118194-0001LF, J3 0475710001, P2 CONNECTOR-15686115148922, U1 V3S, U2 AP65111A, U3 AP65111A, U4 AP65111A, U5 PMIC-LDO-XC6206P302MR(SOT23)

Commit message: added jumpers
Parts:
- removed C46, C73: 4u7, marius:C0603
- removed C47, C74: 47p, marius:C0603
- removed C48, C49, C75, C76: 10u, marius:C0603
- removed IC1: 1V8, AP3410:MCP73811/2
- removed IC3: 1V2, AP3410:MCP73811/2
- removed L4, L8: 2.2uH-DCR<0.1R-1.5A, marius:L4X4
- removed R31, R32, R43: 100K-1%, resistor:R-EU_R0402
- removed R42: 200K-1%, resistor:R-EU_R0402
- removed SJ2, SJ3: (no value), jumper:SJ
- added C54, C58: 4u7, marius:C0603
- added C55, C59: 47p, marius:C0603
- added C56, C57, C60, C61: 10u, marius:C0603
- added IC5, IC6: 3V#, AP3410:MCP73811/2
- added L6, L9: 2.2uH-DCR<0.1R-1.5A, marius:L4X4
- added R35, R36, R38: 100K-1%, resistor:R-EU_R0402
- added R37: 200K-1%, resistor:R-EU_R0402
- added SJ4, SJ5, SJ6, SJ8, SJ9: (no value), jumper:SJ
Connections:
- removed net N$33: IC1.LX, L8.1
- removed net N$37: C74.1, IC1.FB, R42.1, R43.1
- removed net N$7: IC3.LX, L4.1
- removed net N$8: C47.1, IC3.FB, R31.1, R32.1
- new net N$45: IC5.LX, L6.1
- new net N$46: C55.1, IC5.FB, R35.1, R36.1
- new net N$51: IC6.LX, L9.1
- new net N$52: C59.1, IC6.FB, R37.1, R38.1
- new net P1V2: C18.+, C19.1, L3.2, R14.1, SJ6.1
- new net P1V8: C13.+, C14.1, L2.2, R10.1, SJ5.1
- new net P3V3: C8.+, C9.1, L1.2, R6.1, SJ4.1
- new net PRE1V2: C54.2, C55.2, C56.2, L6.2, R35.2, SJ8.1
- new net PRE1V8: C58.2, C59.2, C60.2, L9.2, R37.2, SJ9.1
- new net PRE3V3: C69.2, C70.2, C71.2, L7.2, R40.2, SJ1.1
- net 1V2: now also SJ6.2, SJ8.2; no longer C18.+, C19.1, C46.2, C47.2, C48.2, L3.2, L4.2, R14.1, R31.2
- net 1V8: now also SJ5.2, SJ9.2; no longer C13.+, C14.1, C73.2, C74.2, C75.2, L2.2, L8.2, R10.1, R42.2
- net 3V3: now also SJ1.2, SJ4.2; no longer C69.2, C70.2, C71.2, C8.+, C9.1, L1.2, L7.2, R40.2, R6.1
- net GND: now also C54.1, C56.1, C57.2, C58.1, C60.1, C61.2, IC5.GND, IC6.GND, R36.2, R38.2; no longer C46.1, C48.1, C49.2, C73.1, C75.1, C76.2, IC1.GND, IC3.GND, R32.2, R43.2
- net VCC: now also C57.1, C61.1, IC2.EN, IC5.EN, IC5.VIN, IC6.EN, IC6.VIN; no longer C49.1, C76.1, IC1.VIN, IC3.VIN

Commit message: high
Connections:
- net N$5 renamed USBDIFF_N
- net N$6 renamed USBDIFF_P
- net N$65 renamed D0_N
- net N$66 renamed D0_P
- net N$68 renamed D1_N
- net N$69 renamed D1_P
- net N$70 renamed CK_P
- net N$72 renamed CK_N
Changed lines of the file:
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@@
 </variantdefs>
 <classes>
-<class number="0" name="default" width="0.25" drill="0.35">
+<class number="0" name="default" width="0.2" drill="0.35">
 <clearance class="0" value="0.15"/>
+</class>
+<class number="1" name="diff pairs" width="0.4064" drill="0">
 </class>
 <class number="3" name="power" width="0.35" drill="0.35">
@@
 </segment>
 </net>
-<net name="N$5" class="0">
+<net name="USBDIFF_N" class="1">
 <segment>
 <pinref part="U1" gate="G$5" pin="USB-DM"/>
 <pinref part="J1" gate="G$1" pin="DM"/>
 <wire x1="53.34" y1="96.52" x2="27.94" y2="96.52" width="0.1524" layer="91"/>
-</segment>
-</net>
-<net name="N$6" class="0">
+<label x="40.64" y="96.52" size="1.778" layer="95"/>
+</segment>
+</net>
+<net name="USBDIFF_P" class="1">
 <segment>
 <pinref part="J1" gate="G$1" pin="DP"/>
@@
 <wire x1="27.94" y1="93.98" x2="53.34" y2="93.98" width="0.1524" layer="91"/>
 <wire x1="53.34" y1="93.98" x2="53.34" y2="91.44" width="0.1524" layer="91"/>
+<label x="40.64" y="93.98" size="1.778" layer="95"/>
 </segment>
 </net>
@@
 </segment>
 </net>
-<net name="N$65" class="0">
+<net name="D0_N" class="0">
 <segment>
 <pinref part="P2" gate="G$1" pin="2"/>
@@
 <pinref part="U1" gate="G$3" pin="MCSI-D0N"/>
 <wire x1="119.38" y1="45.72" x2="99.06" y2="45.72" width="0.1524" layer="91"/>
-</segment>
-</net>
-<net name="N$66" class="0">
+<label x="106.68" y="45.72" size="1.778" layer="95"/>
+</segment>
+</net>
+<net name="D0_P" class="0">
 <segment>
 <pinref part="P2" gate="G$1" pin="3"/>
@@
 <wire x1="99.06" y1="50.8" x2="121.92" y2="50.8" width="0.1524" layer="91"/>
 <wire x1="121.92" y1="50.8" x2="121.92" y2="55.88" width="0.1524" layer="91"/>
-</segment>
-</net>
-<net name="N$68" class="0">
+<label x="106.68" y="50.8" size="1.778" layer="95"/>
+</segment>
+</net>
+<net name="D1_N" class="0">
 <segment>
 <pinref part="P2" gate="G$1" pin="5"/>
@@
 <pinref part="U1" gate="G$3" pin="MCSI-D1N"/>
 <wire x1="124.46" y1="35.56" x2="99.06" y2="35.56" width="0.1524" layer="91"/>
-</segment>
-</net>
-<net name="N$69" class="0">
+<label x="106.68" y="35.56" size="1.778" layer="95"/>
+</segment>
+</net>
+<net name="D1_P" class="0">
 <segment>
 <pinref part="U1" gate="G$3" pin="MCSI-D1P"/>
@@
 <pinref part="P2" gate="G$1" pin="6"/>
 <wire x1="127" y1="48.26" x2="144.78" y2="48.26" width="0.1524" layer="91"/>
-</segment>
-</net>
-<net name="N$70" class="0">
+<label x="106.68" y="40.64" size="1.778" layer="95"/>
+</segment>
+</net>
+<net name="CK_P" class="0">
 <segment>
 <pinref part="P2" gate="G$1" pin="8"/>
@@
 <wire x1="60.96" y1="45.72" x2="55.88" y2="45.72" width="0.1524" layer="91"/>
 <wire x1="55.88" y1="45.72" x2="55.88" y2="27.94" width="0.1524" layer="91"/>
-</segment>
-</net>
-<net name="N$72" class="0">
+<label x="106.68" y="27.94" size="1.778" layer="95"/>
+</segment>
+</net>
+<net name="CK_N" class="0">
 <segment>
 <pinref part="U1" gate="G$3" pin="MCSI-CKP"/>
@@
 <pinref part="P2" gate="G$1" pin="9"/>
 <wire x1="134.62" y1="40.64" x2="144.78" y2="40.64" width="0.1524" layer="91"/>
-</segment>
-</net>
+<label x="106.68" y="22.86" size="1.778" layer="95"/>
+</segment>
+</net>

Commit message: In progress
Parts:
- R16: device marius:R0603 -> marius:R0402
Connections:
- new net LEDD0: R45.1
- new net LEDD1: R46.1
- net LED0: no longer R45.1
- net LED1: no longer R46.1

Commit message: In progress
Parts:
- removed C43: 10u, marius:C0603
- renumbered C40 to 3V3
Connections:
- net 3V3: no longer C43.1
- net GND: no longer C43.2
Changed lines of the file:
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@@
 <part name="C38" library="marius" library_urn="urn:adsk.eagle:library:5910807" deviceset="C" device="0603" package3d_urn="urn:adsk.eagle:package:5911006/1" value="10u"/>
 <part name="C39" library="marius" library_urn="urn:adsk.eagle:library:5910807" deviceset="C" device="0603" package3d_urn="urn:adsk.eagle:package:5911006/1" value="10u"/>
-<part name="C40" library="marius" library_urn="urn:adsk.eagle:library:5910807" deviceset="C" device="0603" package3d_urn="urn:adsk.eagle:package:5911006/1" value="10u"/>
+<part name="3V3" library="marius" library_urn="urn:adsk.eagle:library:5910807" deviceset="C" device="0603" package3d_urn="urn:adsk.eagle:package:5911006/1" value="10u"/>
 <part name="C41" library="marius" library_urn="urn:adsk.eagle:library:5910807" deviceset="C" device="0603" package3d_urn="urn:adsk.eagle:package:5911006/1" value="10u"/>
 <part name="C42" library="marius" library_urn="urn:adsk.eagle:library:5910807" deviceset="C" device="0603" package3d_urn="urn:adsk.eagle:package:5911006/1" value="10u"/>
-<part name="C43" library="marius" library_urn="urn:adsk.eagle:library:5910807" deviceset="C" device="0603" package3d_urn="urn:adsk.eagle:package:5911006/1" value="10u"/>
 <part name="C44" library="marius" library_urn="urn:adsk.eagle:library:5910807" deviceset="C" device="0603" package3d_urn="urn:adsk.eagle:package:5911006/1" value="10u"/>
 <part name="C45" library="marius" library_urn="urn:adsk.eagle:library:5910807" deviceset="C" device="0603" package3d_urn="urn:adsk.eagle:package:5911006/1" value="10u"/>
@@
 <attribute name="VALUE" x="176.784" y="152.781" size="1.778" layer="96"/>
 </instance>
-<instance part="C40" gate="G$1" x="180.34" y="157.48" smashed="yes">
+<instance part="3V3" gate="G$1" x="180.34" y="157.48" smashed="yes">
 <attribute name="NAME" x="181.864" y="157.861" size="1.778" layer="95"/>
 <attribute name="VALUE" x="181.864" y="152.781" size="1.778" layer="96"/>
@@
 <attribute name="NAME" x="192.024" y="157.861" size="1.778" layer="95"/>
 <attribute name="VALUE" x="192.024" y="152.781" size="1.778" layer="96"/>
-</instance>
-<instance part="C43" gate="G$1" x="195.58" y="157.48" smashed="yes">
-<attribute name="NAME" x="197.104" y="157.861" size="1.778" layer="95"/>
-<attribute name="VALUE" x="197.104" y="152.781" size="1.778" layer="96"/>
 </instance>
 <instance part="C44" gate="G$1" x="200.66" y="157.48" smashed="yes">
@@
 <wire x1="175.26" y1="160.02" x2="180.34" y2="160.02" width="0.1524" layer="91"/>
 <junction x="175.26" y="160.02"/>
-<pinref part="C40" gate="G$1" pin="1"/>
+<pinref part="3V3" gate="G$1" pin="1"/>
 <wire x1="180.34" y1="160.02" x2="185.42" y2="160.02" width="0.1524" layer="91"/>
 <junction x="180.34" y="160.02"/>
@@
 <junction x="185.42" y="160.02"/>
 <pinref part="C42" gate="G$1" pin="1"/>
-<wire x1="190.5" y1="160.02" x2="195.58" y2="160.02" width="0.1524" layer="91"/>
 <junction x="190.5" y="160.02"/>
-<pinref part="C43" gate="G$1" pin="1"/>
-<wire x1="195.58" y1="160.02" x2="200.66" y2="160.02" width="0.1524" layer="91"/>
-<junction x="195.58" y="160.02"/>
+<wire x1="190.5" y1="160.02" x2="200.66" y2="160.02" width="0.1524" layer="91"/>
 <pinref part="C44" gate="G$1" pin="1"/>
 <wire x1="200.66" y1="160.02" x2="205.74" y2="160.02" width="0.1524" layer="91"/>
@@
 <wire x1="175.26" y1="152.4" x2="180.34" y2="152.4" width="0.1524" layer="91"/>
 <junction x="175.26" y="152.4"/>
-<pinref part="C40" gate="G$1" pin="2"/>
+<pinref part="3V3" gate="G$1" pin="2"/>
 <wire x1="180.34" y1="152.4" x2="185.42" y2="152.4" width="0.1524" layer="91"/>
 <junction x="180.34" y="152.4"/>
@@
 <wire x1="185.42" y1="152.4" x2="190.5" y2="152.4" width="0.1524" layer="91"/>
 <junction x="185.42" y="152.4"/>
-<wire x1="190.5" y1="152.4" x2="195.58" y2="152.4" width="0.1524" layer="91"/>
 <junction x="190.5" y="152.4"/>
-<pinref part="C43" gate="G$1" pin="2"/>
 <pinref part="C45" gate="G$1" pin="2"/>
-<wire x1="195.58" y1="152.4" x2="200.66" y2="152.4" width="0.1524" layer="91"/>
+<wire x1="190.5" y1="152.4" x2="200.66" y2="152.4" width="0.1524" layer="91"/>
 <pinref part="C44" gate="G$1" pin="2"/>
 <wire x1="200.66" y1="152.4" x2="205.74" y2="152.4" width="0.1524" layer="91"/>
@@
 <junction x="205.74" y="152.4"/>
 <junction x="165.1" y="152.4"/>
-<wire x1="195.58" y1="152.4" x2="165.1" y2="152.4" width="0.1524" layer="91"/>
-<wire x1="195.58" y1="152.4" x2="205.74" y2="152.4" width="0.1524" layer="91"/>
-<junction x="195.58" y="152.4"/>
+<wire x1="205.74" y1="152.4" x2="165.1" y2="152.4" width="0.1524" layer="91"/>
 <label x="185.42" y="152.4" size="1.778" layer="95" rot="R270"/>
 </segment>

Commit message: in progress
Connections:
- removed net N$57: PWM0.2, U1G$2.PB4/PWM0
- removed net N$58: PWM1.2, U1G$2.PB5/PWM1
- net LEDD0: now also PWM0.2, U1G$2.PB4/PWM0
- net LEDD1: now also PWM1.2, U1G$2.PB5/PWM1
Changed lines of the file:
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@@
 </variantdefs>
 <classes>
-<class number="0" name="default" width="0.25" drill="0.35">
+<class number="0" name="default" width="0.2" drill="0.35">
 <clearance class="0" value="0.15"/>
 </class>
@@
 <clearance class="1" value="0.1"/>
 </class>
-<class number="3" name="power" width="0.35" drill="0.35">
+<class number="3" name="power" width="0.25" drill="0.35">
 <clearance class="3" value="0.15"/>
 </class>
@@
 </segment>
 </net>
-<net name="N$57" class="0">
+<net name="LEDD0" class="0">
 <segment>
 <pinref part="U1" gate="G$2" pin="PB4/PWM0"/>
 <wire x1="116.84" y1="83.82" x2="121.92" y2="83.82" width="0.1524" layer="91"/>
 <pinref part="PWM0" gate="G$1" pin="2"/>
-</segment>
-</net>
-<net name="N$58" class="0">
+<label x="121.92" y="83.82" size="1.778" layer="95" rot="R90"/>
+</segment>
+</net>
+<net name="LEDD1" class="0">
 <segment>
 <pinref part="U1" gate="G$2" pin="PB5/PWM1"/>
 <wire x1="116.84" y1="78.74" x2="121.92" y2="78.74" width="0.1524" layer="91"/>
 <pinref part="PWM1" gate="G$1" pin="2"/>
+<label x="121.92" y="78.74" size="1.778" layer="95" rot="R90"/>
 </segment>
 </net>
@@
 </segment>
 </net>
-<net name="N$13" class="3">
+<net name="N$13" class="0">
 <segment>
 <pinref part="U1" gate="G$6" pin="VCC-RTC"/>

Commit message: In Progress
Parts:
- added C40, C43, C46: 10u, marius:C0603
- added CLK, INT, RST, WOL: TEST_TESTPOINT, marius:TEST_TESTPOINT
- added J2: CONNECTOR-10HEADER-5X2, marius:CONNECTOR-10HEADER-5X2
- added J4: CONNECTOR-4HEADER4, marius:CONNECTOR-4HEADER4
- added J5: CONNECTOR-3HEADER3, marius:CONNECTOR-3HEADER3
- added R31: 10k, resistor:R-EU_R0402
- D1, D2, D3: MPN (none) -> HQ67-23A2ARGBC
- IC2: MPN (none) -> AP3410KTR-G1
- IC6: value 3V# -> MCP73811/2; MPN (none) -> AP3410KTR-G1
- L6, L7, L9: MOUSER (none) -> LVF404018-2R2M-N; MPN (none) -> LVF404018-2R2M-N
- X1: MPN (none) -> 7U24000E09UCG
- X2: MPN (none) -> SF32K32768D71T01
Connections:
- removed net N$53: MISO.2, U1G$2.PC0/SPI1/MISO
- removed net N$54: SCK.2, U1G$2.PC1/SPI1/SCK
- removed net N$55: CS.2, U1G$2.PC2/SPI1/CS
- removed net N$56: MOSI.2, U1G$2.PC3/SPI1/MOSI
- new net CLK: CLK.2, J2.10
- new net CS: CS.2, J2.4, R31.2, U1G$2.PC2/SPI1/CS
- new net INT: INT.2, J2.9
- new net MISO: J2.7, MISO.2, U1G$2.PC0/SPI1/MISO
- new net MOSI: J2.6, MOSI.2, U1G$2.PC3/SPI1/MOSI
- new net RST: J2.3, RST.2
- new net SCK: J2.5, SCK.2, U1G$2.PC1/SPI1/SCK
- new net WOL: J2.8, WOL.2
- net 3V3: now also C43.1, J2.2, R31.1
- net GND: now also C40.1, C43.2, C46.1, J2.1, J4.1, J5.1
- net LEDD0: now also J5.2
- net SCL: now also J4.3
- net SDA: now also J4.4
- net VCC: now also C40.2, C46.2, J4.2, J5.3
Other:
- moved on the sheet: CAMIO0, CAMIO1

Commit message: In progress
Parts:
- added C47, C48: 10u, marius:C0603
- added J6: HR911105A, HR911105A:HR911105A
- added L4: 10uH(NC), marius:L0603
- added R32, R33, R34, R39: 51(NC), resistor:R-EU_R0402
- added R42: 6K-1%, resistor:R-EU_R0402
Connections:
- new net ETH_RX_N: J6.RD-, R34.1, U1G$5.EPHY_RXN
- new net ETH_RX_P: J6.RD+, R33.1, U1G$5.EPHY_RXP
- new net ETH_TX_N: J6.TD-, R39.1, U1G$5.EPHY_TXN
- new net ETH_TX_P: J6.TD+, R32.1, U1G$5.EPHY_TXP
- new net N$37: R42.2, U1G$5.EPHY_RTX
- new net N$55: C47.1, J6.P4, R32.2, R39.2
- new net N$56: C48.1, J6.P5, L4.2, R33.2, R34.2
- net 3V3: now also C40.2, J4.2, L4.1
- net GND: now also C47.2, C48.2, J6.GC, J6.GND, J6.SHIELD, J6.YC, R42.1
- net LED3: now also J6.GA
- net LED4: now also J6.YA
- net VCC: no longer C40.2, J4.2
Other:
- moved on the sheet: FID1, FID2
